File: pcb/PCB.kicad_pcb (KiCad board)
At the start: 4 copper layers, 29.2 x 51.1 mm, 35 parts, among them J1 Conn_01x15, J2 USB_C_Receptacle_USB2.0, J3 Conn_01x15, J4 TC2030, J5 Conn_01x04, SW1 SW_Push, SW2 SW_Push, U1 SN65HVD230, U2 AMS1117-3.3, U3 STM32F103C8T6, Y1 8MHz

Commit message: Finished schematic
Parts:
- removed FB2: 100R@100MHz, Resistor_SMD:R_0805_2012Metric
- removed J4: TC2030, Connector:Tag-Connect_TC2030-IDC-NL_2x03_P1.27mm_Vertical
- removed J5: Conn_01x04, Connector_PinHeader_2.54mm:PinHeader_1x04_P2.54mm_Vertical
- removed JP1: SolderJumper_Bridged, Jumper:SolderJumper-2_P1.3mm_Bridged_RoundedPad1.0x1.5mm
- added C13: 100n, Capacitor_SMD:C_0402_1005Metric, F.Cu at (371.6, 149.7)
- added C14: 100n, Capacitor_SMD:C_0402_1005Metric, F.Cu at (380.1, 142.2)
- added C15: 1u, Capacitor_SMD:C_0603_1608Metric, F.Cu at (376.4, 145.5)
- added C16: 100n, Capacitor_SMD:C_0402_1005Metric, F.Cu at (379.8, 144.8)
- added C17: 220p, Capacitor_SMD:C_0402_1005Metric, F.Cu at (389.4, 98.6)
- added C18: 100nF >25V, Capacitor_SMD:C_0805_2012Metric, F.Cu at (366.8, 100.1)
- added C19: 10nF >25V, Capacitor_SMD:C_0805_2012Metric, F.Cu at (363.3, 100.1)
- added C20: 2.2uF, Capacitor_SMD:C_0805_2012Metric, F.Cu at (247.1, 73.2)
- added C21: 100nF, Capacitor_SMD:C_0603_1608Metric, F.Cu at (247.1, 75.7)
- added C22: 2.2uF, Capacitor_SMD:C_0805_2012Metric, F.Cu at (258.6, 73.2)
- added C23: 100nF, Capacitor_SMD:C_0603_1608Metric, F.Cu at (258.6, 75.7)
- added C24: 2.2uF, Capacitor_SMD:C_0805_2012Metric, F.Cu at (270.0, 73.2)
- added C25: 100nF, Capacitor_SMD:C_0603_1608Metric, F.Cu at (270.0, 75.7)
- added C26: 2.2uF, Capacitor_SMD:C_0805_2012Metric, F.Cu at (281.4, 73.2)
- added C27: 100nF, Capacitor_SMD:C_0603_1608Metric, F.Cu at (281.4, 75.7)
- added C28: 2.2uF, Capacitor_SMD:C_0805_2012Metric, F.Cu at (292.9, 73.2)
- added C29: 100nF, Capacitor_SMD:C_0603_1608Metric, F.Cu at (292.9, 75.7)
- added C30: 2.2uF, Capacitor_SMD:C_0805_2012Metric, F.Cu at (304.3, 73.2)
- added C31: 100nF, Capacitor_SMD:C_0603_1608Metric, F.Cu at (304.3, 75.7)
- added C32: 220p, Capacitor_SMD:C_0402_1005Metric, F.Cu at (223.4, 319.1)
- added C33: 100nF >25V, Capacitor_SMD:C_0805_2012Metric, F.Cu at (460.8, 128.3)
- added C34: 10nF >25V, Capacitor_SMD:C_0805_2012Metric, F.Cu at (469.4, 121.9)
- added C35: 220p, Capacitor_SMD:C_0402_1005Metric, F.Cu at (432.5, 261.2)
- added C36: 100nF >25V, Capacitor_SMD:C_0805_2012Metric, F.Cu at (480.8, 128.3)
- added C37: 10nF >25V, Capacitor_SMD:C_0805_2012Metric, F.Cu at (489.3, 121.9)
- added C38: 220p, Capacitor_SMD:C_0402_1005Metric, F.Cu at (340.5, 259.8)
- added C39: 100nF >25V, Capacitor_SMD:C_0805_2012Metric, F.Cu at (480.8, 115.8)
- added C40: 10nF >25V, Capacitor_SMD:C_0805_2012Metric, F.Cu at (489.3, 109.4)
- added C41: 220p, Capacitor_SMD:C_0402_1005Metric, F.Cu at (223.4, 276.5)
- added C42: 100nF >25V, Capacitor_SMD:C_0805_2012Metric, F.Cu at (460.8, 115.8)
- added C43: 10nF >25V, Capacitor_SMD:C_0805_2012Metric, F.Cu at (469.4, 109.4)
- added C44: 220p, Capacitor_SMD:C_0402_1005Metric, F.Cu at (432.5, 218.7)
- added C45: 100nF >25V, Capacitor_SMD:C_0805_2012Metric, F.Cu at (460.8, 140.8)
- added C46: 10nF >25V, Capacitor_SMD:C_0805_2012Metric, F.Cu at (469.4, 134.4)
- added D10: SSB43L, Diode_SMD:D_SMB, F.Cu at (305.6, 102.4)
- added D11: 7V, Diode_SMD:D_MiniMELF, F.Cu at (226.6, 320.3)
- added D12: 7V, Diode_SMD:D_MiniMELF, F.Cu at (435.7, 262.5)
- added D13: 7V, Diode_SMD:D_MiniMELF, F.Cu at (339.2, 263.0)
- added D14: 7V, Diode_SMD:D_MiniMELF, F.Cu at (226.6, 277.8)
- added D15: 7V, Diode_SMD:D_MiniMELF, F.Cu at (435.7, 219.9)
- added D16: SP0502BAHT, Package_TO_SOT_SMD:SOT-23, F.Cu at (353.6, 135.7)
- added D3: ESDCAN02-2BWY, Package_TO_SOT_SMD:SOT-23, F.Cu at (248.7, 184.5)
- added D4: 7V, Diode_SMD:D_MiniMELF, F.Cu at (386.2, 97.3)
- added D5: SSB43L, Diode_SMD:D_SMB, F.Cu at (248.4, 102.4)
- added D6: SSB43L, Diode_SMD:D_SMB, F.Cu at (259.8, 102.4)
- added D7: SSB43L, Diode_SMD:D_SMB, F.Cu at (271.3, 102.4)
- added D8: SSB43L, Diode_SMD:D_SMB, F.Cu at (282.7, 102.4)
- added D9: SSB43L, Diode_SMD:D_SMB, F.Cu at (294.1, 102.4)
- added F1: Fuse, Fuse:Fuseholder_Blade_Mini_Keystone_3568, F.Cu at (247.6, 112.6)
- added F2: Fuse, Fuse:Fuseholder_Blade_Mini_Keystone_3568, F.Cu at (255.2, 112.6)
- added F3: Fuse, Fuse:Fuseholder_Blade_Mini_Keystone_3568, F.Cu at (262.8, 112.6)
- added F4: Fuse, Fuse:Fuseholder_Blade_Mini_Keystone_3568, F.Cu at (270.4, 112.6)
- added F5: Fuse, Fuse:Fuseholder_Blade_Mini_Keystone_3568, F.Cu at (278.1, 112.6)
- added F6: Fuse, Fuse:Fuseholder_Blade_Mini_Keystone_3568, F.Cu at (285.7, 112.6)
- added Q1: IRLZ44N, Package_TO_SOT_SMD:TO-263-2, F.Cu at (247.1, 91.4)
- added Q2: IRLZ44N, Package_TO_SOT_SMD:TO-263-2, F.Cu at (258.6, 91.4)
- added Q3: IRLZ44N, Package_TO_SOT_SMD:TO-263-2, F.Cu at (270.0, 91.4)
- added Q4: IRLZ44N, Package_TO_SOT_SMD:TO-263-2, F.Cu at (281.4, 91.4)
- added Q5: IRLZ44N, Package_TO_SOT_SMD:TO-263-2, F.Cu at (292.9, 91.4)
- added Q6: IRLZ44N, Package_TO_SOT_SMD:TO-263-2, F.Cu at (304.3, 91.4)
- added R10: 4.7k, Resistor_SMD:R_0603_1608Metric, F.Cu at (244.6, 77.0)
- added R11: 4.7k, Resistor_SMD:R_0603_1608Metric, F.Cu at (256.0, 77.0)
- added R12: 4.7k, Resistor_SMD:R_0603_1608Metric, F.Cu at (267.5, 77.0)
- added R13: 4.7k, Resistor_SMD:R_0603_1608Metric, F.Cu at (278.9, 77.0)
- added R14: 4.7k, Resistor_SMD:R_0603_1608Metric, F.Cu at (290.3, 77.0)
- added R15: 4.7k, Resistor_SMD:R_0603_1608Metric, F.Cu at (301.8, 77.0)
- added R16: 4.7k, Resistor_SMD:R_0603_1608Metric, F.Cu at (223.4, 321.6)
- added R17: 4.7k, Resistor_SMD:R_0603_1608Metric, F.Cu at (469.1, 128.1)
- added R18: 4.7k, Resistor_SMD:R_0603_1608Metric, F.Cu at (229.7, 321.6)
- added R19: 4.7k, Resistor_SMD:R_0603_1608Metric, F.Cu at (465.1, 128.1)
- added R20: 1.2k, Resistor_SMD:R_0603_1608Metric, F.Cu at (229.7, 319.1)
- added R21: 47, Resistor_SMD:R_0603_1608Metric, F.Cu at (469.2, 124.6)
- added R22: 4.7k, Resistor_SMD:R_0603_1608Metric, F.Cu at (432.5, 263.8)
- added R23: 4.7k, Resistor_SMD:R_0603_1608Metric, F.Cu at (489.0, 128.1)
- added R24: 4.7k, Resistor_SMD:R_0603_1608Metric, F.Cu at (438.8, 263.8)
- added R25: 4.7k, Resistor_SMD:R_0603_1608Metric, F.Cu at (485.0, 128.1)
- added R26: 1.2k, Resistor_SMD:R_0603_1608Metric, F.Cu at (438.8, 261.2)
- added R27: 47, Resistor_SMD:R_0603_1608Metric, F.Cu at (489.1, 124.6)
- added R28: 4.7k, Resistor_SMD:R_0603_1608Metric, F.Cu at (337.9, 259.8)
- added R29: 4.7k, Resistor_SMD:R_0603_1608Metric, F.Cu at (489.0, 115.6)
- added R30: 4.7k, Resistor_SMD:R_0603_1608Metric, F.Cu at (337.9, 266.2)
- added R31: 4.7k, Resistor_SMD:R_0603_1608Metric, F.Cu at (485.0, 115.6)
- added R32: 1.2k, Resistor_SMD:R_0603_1608Metric, F.Cu at (340.5, 266.2)
- added R33: 47, Resistor_SMD:R_0603_1608Metric, F.Cu at (489.1, 112.1)
- added R34: 4.7k, Resistor_SMD:R_0603_1608Metric, F.Cu at (223.4, 279.0)
- added R35: 4.7k, Resistor_SMD:R_0603_1608Metric, F.Cu at (469.1, 115.6)
- added R36: 4.7k, Resistor_SMD:R_0603_1608Metric, F.Cu at (229.7, 279.0)
- added R37: 4.7k, Resistor_SMD:R_0603_1608Metric, F.Cu at (465.1, 115.6)
- added R38: 1.2k, Resistor_SMD:R_0603_1608Metric, F.Cu at (229.7, 276.5)
- added R39: 47, Resistor_SMD:R_0603_1608Metric, F.Cu at (469.2, 112.1)
- added R40: 4.7k, Resistor_SMD:R_0603_1608Metric, F.Cu at (432.5, 221.2)
- added R41: 4.7k, Resistor_SMD:R_0603_1608Metric, F.Cu at (469.1, 140.6)
- added R42: 4.7k, Resistor_SMD:R_0603_1608Metric, F.Cu at (438.8, 221.2)
- added R43: 4.7k, Resistor_SMD:R_0603_1608Metric, F.Cu at (465.1, 140.6)
- added R44: 1.2k, Resistor_SMD:R_0603_1608Metric, F.Cu at (438.8, 218.7)
- added R45: 47, Resistor_SMD:R_0603_1608Metric, F.Cu at (469.2, 137.2)
- added R46: 470, Resistor_SMD:R_0603_1608Metric, F.Cu at (342.7, 149.4)
- added R8: 1.2k, Resistor_SMD:R_0603_1608Metric, F.Cu at (383.0, 98.6)
- added R9: 47, Resistor_SMD:R_0603_1608Metric, F.Cu at (371.6, 99.4)
- added U10: MCP1416, Package_TO_SOT_SMD:SOT-23-5, F.Cu at (304.3, 79.5)
- added U11: BTS7004-1EPP, Package_SO:Infineon_PG-TSDSO-14-22, F.Cu at (462.9, 123.6)
- added U12: BTS7004-1EPP, Package_SO:Infineon_PG-TSDSO-14-22, F.Cu at (482.8, 123.6)
- added U13: BTS7004-1EPP, Package_SO:Infineon_PG-TSDSO-14-22, F.Cu at (482.8, 111.1)
- added U14: BTS7004-1EPP, Package_SO:Infineon_PG-TSDSO-14-22, F.Cu at (462.9, 111.1)
- added U15: BTS7004-1EPP, Package_SO:Infineon_PG-TSDSO-14-22, F.Cu at (462.9, 136.1)
- added U4: BTS7004-1EPP, Package_SO:Infineon_PG-TSDSO-14-22, F.Cu at (365.9, 96.3)
- added U5: MCP1416, Package_TO_SOT_SMD:SOT-23-5, F.Cu at (247.1, 79.5)
- added U6: MCP1416, Package_TO_SOT_SMD:SOT-23-5, F.Cu at (258.6, 79.5)
- added U7: MCP1416, Package_TO_SOT_SMD:SOT-23-5, F.Cu at (270.0, 79.5)
- added U8: MCP1416, Package_TO_SOT_SMD:SOT-23-5, F.Cu at (281.4, 79.5)
- added U9: MCP1416, Package_TO_SOT_SMD:SOT-23-5, F.Cu at (292.9, 79.5)
- C11: value 1u -> 30p; footprint Capacitor_SMD:C_0603_1608Metric -> Capacitor_SMD:C_0402_1005Metric
- C2: value 1u -> 100uF; footprint Capacitor_SMD:C_0603_1608Metric -> Capacitor_SMD:CP_Elec_6.3x7.7
- C3: value 1u -> 2.2uF; footprint Capacitor_SMD:C_0603_1608Metric -> Capacitor_SMD:C_0805_2012Metric
- C4: value 4u7 -> 100nF
- C5: value 30p -> 100uF; footprint Capacitor_SMD:C_0402_1005Metric -> Capacitor_SMD:CP_Elec_6.3x7.7
- C7: value 30p -> 100nF; footprint Capacitor_SMD:C_0402_1005Metric -> Capacitor_SMD:C_0603_1608Metric
- C8: value 100n -> 4u7; footprint Capacitor_SMD:C_0402_1005Metric -> Capacitor_SMD:C_0603_1608Metric
- C9: value 100n -> 30p
- D1: value YELLOW -> 15-25V; footprint LED_SMD:LED_0603_1608Metric -> Diode_SMD:D_SMA
- D2: value BLUE -> SP0502BAHT; footprint LED_SMD:LED_0603_1608Metric -> Package_TO_SOT_SMD:SOT-23
- J1: value Conn_01x15 -> DTM1312PA12PBR008; footprint Connector_PinHeader_2.54mm:PinHeader_1x15_P2.54mm_Vertical -> DTM13-12PA-12PB:TE_DTM1312PA12PBR008
- J2: value USB_C_Receptacle_USB2.0 -> TC2030; footprint Connector_USB:USB_C_Receptacle_HRO_TYPE-C-31-M-12 -> Connector:Tag-Connect_TC2030-IDC-NL_2x03_P1.27mm_Vertical
- J3: value Conn_01x15 -> Conn_02x08_Top_Bottom; footprint Connector_PinHeader_2.54mm:PinHeader_1x15_P2.54mm_Vertical -> Connector_PinHeader_2.54mm:PinHeader_2x08_P2.54mm_Vertical
- R1, R2: value 5k1 -> 470; footprint Resistor_SMD:R_0402_1005Metric -> Resistor_SMD:R_0603_1608Metric
- R3: value 120R -> 5k1; footprint Resistor_SMD:R_0402_1005Metric -> Resistor_SMD:R_0603_1608Metric
- R4, R6, R7: value 1k5 -> 4.7k; footprint Resistor_SMD:R_0402_1005Metric -> Resistor_SMD:R_0603_1608Metric
- R5: value 5k1 -> 4.7k; footprint Resistor_SMD:R_0402_1005Metric -> Resistor_SMD:R_0603_1608Metric
- moved Y1 253.5 mm to (394.1, 135.9), turned to 0 degrees
- moved SW2 253.1 mm to (385.4, 137.4), turned to 0 degrees
- moved C10 241.0 mm to (391.9, 139.3), turned to 0 degrees
- moved FB1 237.8 mm to (372.4, 142.7), turned to 0 degrees
- moved J2 236.9 mm to (367.0, 169.8), turned to 0 degrees
- moved R4 236.3 mm to (389.4, 96.0), turned to 180 degrees
- moved R6 235.6 mm to (383.0, 96.0), turned to 0 degrees
- moved C9 234.8 mm to (371.6, 147.7), turned to 0 degrees
- moved C11 233.9 mm to (374.5, 149.7), turned to 0 degrees
- moved C12 232.8 mm to (374.5, 147.7), turned to 0 degrees
- moved R7 232.6 mm to (371.6, 97.5), turned to 180 degrees
- moved U3 228.4 mm to (368.7, 161.6), turned to 0 degrees
- moved R3 228.2 mm to (376.6, 142.5)
- moved C8 227.0 mm to (372.2, 145.5), turned to 0 degrees
- moved SW1 226.0 mm to (375.3, 137.4), turned to 0 degrees
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Connections:
- net /NRST renamed /STM32/NRST
- C11 pad 1: +3.3VA -> /STM32/HSE_IN
- C12 pad 1: +3.3VA -> +3V3
- C2 pad 1: VCC -> +12V
- C3 pad 1: +3V3 -> +12V
- C4 pad 1: +3V3 -> +12V
- C5 pad 1: /HSE_OUT -> +3V3
- C6 pad 1: +3V3 -> Net-(C6-Pad1)
- C6 pad 2: GND -> Net-(C6-Pad2)
- C7 pad 1: /HSE_IN -> +3V3
- C9 pad 1: +3V3 -> /STM32/HSE_OUT
- D1 pad 1: Net-(D1-Pad1) -> +12V
- D1 pad 2: +3V3 -> GND
- D2 pad 1: Net-(D2-Pad1) -> UART_TX
- D2 pad 2: /LED_STAT -> UART_RX
- FB1 pad 1: /VBUS -> +3V3
- FB1 pad 2: VCC -> +3.3VA
- J3 pad 1: +3V3 -> /STM32/UU0
- J3 pad 10: PB0 -> /STM32/UU7
- J3 pad 11: PA7 -> /STM32/UU8
- J3 pad 12: PA6 -> GND
- J3 pad 13: PA5 -> /STM32/UART_RX
- J3 pad 14: PA4 -> /STM32/UART_TX
- J3 pad 15: PA3 -> GND
- J3 pad 2: GND -> /STM32/UU1
- J3 pad 3: PA10 -> /STM32/UU2
- J3 pad 4: PA9 -> /STM32/UU3
- J3 pad 5: PA8 -> /STM32/UU4
- J3 pad 6: PB11 -> /STM32/UU5
- J3 pad 7: PB10 -> GND
- J3 pad 8: PB2 -> +3V3
- J3 pad 9: PB1 -> /STM32/UU6
- R1 pad 1: Net-(J2-PadA5) -> UART_TX
- R1 pad 2: GND -> /STM32/UART_TX
- R2 pad 1: GND -> /STM32/UART_RX
- R2 pad 2: Net-(J2-PadB5) -> UART_RX
- R3 pad 1: /CAN+ -> /STM32/BOOT0
- R3 pad 2: Net-(JP1-Pad2) -> GND
- R4 pad 1: Net-(D1-Pad1) -> /High-side Channel 0/Sense
- R4 pad 2: GND -> Net-(D4-Pad1)
- R5 pad 1: /BOOT0 -> /High-side Channel 0/DEN
- R5 pad 2: GND -> Net-(R5-Pad2)
- R6 pad 1: +3V3 -> Net-(R6-Pad1)
- R6 pad 2: USB_D+ -> Net-(D4-Pad1)
- R7 pad 1: Net-(D2-Pad1) -> /High-side Channel 0/Drive
- R7 pad 2: GND -> Net-(R7-Pad2)
- SW1 pad 1: /BOOT0 -> /STM32/BOOT0
- U1 pad 5: unconnected-(U1-Pad5) -> Net-(C6-Pad1)
- U1 pad 6: /CAN- -> CAN-
- U1 pad 7: /CAN+ -> CAN+
- U2 pad 3: VCC -> +12V
- U3 pad 10: PA0 -> /High-side Channel 0/Sense
- U3 pad 11: /LED_STAT -> /High-side Channel 1/Sense
- U3 pad 12: PA2 -> /High-side Channel 2/Sense
- U3 pad 13: PA3 -> /High-side Channel 3/Sense
- U3 pad 14: PA4 -> /High-side Channel 4/Sense
- U3 pad 15: PA5 -> /High-side Channel 5/Sense
- U3 pad 16: PA6 -> /High-side Channel 0/Drive
- U3 pad 17: PA7 -> /High-side Channel 1/Drive
- U3 pad 18: PB0 -> /High-side Channel 2/Drive
- U3 pad 19: PB1 -> /High-side Channel 3/Drive
- U3 pad 2: PC13 -> /STM32/UU5
- U3 pad 20: PB2 -> /High-side Channel 4/Drive
- U3 pad 21: PB10 -> /Low-side channel 0/Drive
- U3 pad 22: PB11 -> /Low-side channel 1/Drive
- U3 pad 25: unconnected-(U3-Pad25) -> /STM32/GPIO
- U3 pad 26: unconnected-(U3-Pad26) -> /STM32/UU2
- U3 pad 27: unconnected-(U3-Pad27) -> /STM32/UU3
- U3 pad 28: unconnected-(U3-Pad28) -> /STM32/UU4
- U3 pad 29: PA8 -> /Low-side channel 2/Drive
- U3 pad 3: PC14 -> /STM32/UU6
- U3 pad 30: PA9 -> /Low-side channel 3/Drive
- U3 pad 31: PA10 -> /Low-side channel 4/Drive
- U3 pad 32: USB_D- -> /Low-side channel 5/Drive
- U3 pad 33: USB_D+ -> /STM32/UU0
- U3 pad 38: PA15 -> /STM32/UU1
- U3 pad 4: PC15 -> /STM32/UU7
- U3 pad 40: PB4 -> /High-side Channel 5/Drive
- U3 pad 41: PB5 -> /High-side Channel 0/DEN
- U3 pad 42: PB6 -> /STM32/UART_RX
- U3 pad 43: PB7 -> /STM32/UART_TX
- U3 pad 44: /BOOT0 -> /STM32/BOOT0
- U3 pad 5: /HSE_OUT -> /STM32/HSE_OUT
- U3 pad 6: /HSE_IN -> /STM32/HSE_IN
- Y1 pad 1: /HSE_OUT -> /STM32/HSE_OUT
- Y1 pad 2: /HSE_IN -> /STM32/HSE_IN
Routing:
- net +3V3: track 44.0 -> 0.00 mm, vias 18 -> 0
- net GND: track 41.4 -> 2.61 mm, vias 23 -> 1
- net /STM32/NRST: track 35.9 -> 0.00 mm, vias 3 -> 0
- net /BOOT0: track 31.5 -> 0.00 mm, vias 3 -> 0
- net SWDIO: track 24.1 -> 0.00 mm, vias 2 -> 0
- net SWO: track 22.9 -> 0.00 mm, vias 2 -> 0
- net USB_D-: track 21.7 -> 0.00 mm
- net USB_D+: track 21.3 -> 0.00 mm
- net PA2: track 20.8 -> 0.00 mm
- net +3.3VA: track 20.2 -> 0.00 mm, vias 2 -> 0
- net SWCLK: track 19.4 -> 0.00 mm, vias 2 -> 0
- net PA0: track 18.4 -> 0.00 mm
- net /LED_STAT: track 18.2 -> 0.00 mm, vias 2 -> 0
- net PA3: track 18.0 -> 0.00 mm, vias 1 -> 0
- net PB7: track 16.5 -> 0.00 mm
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- added copper zone on B.Cu, net +12V
- added copper zone on F.Cu, net +12V
- added copper zone on F.Cu, net H0
- removed copper zone on In2.Cu, net +3V3
- removed copper zone on B.Cu, net GND
- removed copper zone on In1.Cu, net GND
- removed copper zone on F.Cu, net unconnected-(J2-PadS1)
Other:
- board outline removed
- board text removed: "3V3"
- board text removed: "3V3 +CAN- GND"
- board text removed: "A0"
- board text removed: "A10"
- board text removed: "A13"
- board text removed: "A14"
- board text removed: "A15"
- board text removed: "A2"
- board text removed: "A3"
- board text removed: "A4"
- board text removed: "A5"
- board text removed: "A6"
- board text removed: "A7"
- board text removed: "A8"
- board text removed: "A9"
- board text removed: "B0"
- board text removed: "B1"
- board text removed: "B10"
- board text removed: "B11"
- board text removed: "B2"
- board text removed: "B3"
- board text removed: "B4"
- board text removed: "B5"
- board text removed: "B6"
- board text removed: "B7"
- board text removed: "BOOT"
- board text removed: "C13"
- board text removed: "C14"
- board text removed: "C15"
- board text removed: "CAN TERM"
- board text removed: "GND"
- board text removed: "GND -CAN+ 3V3"
- board text removed: "JLCJLCJLCJLC"
- board text removed: "RESET"
- board text removed: "Rev 1"
- board text removed: "STM32F103 CAN/USB-C Jack LeFevre July 2022"
- board text removed: "SWCLK"
- board text removed: "SWDIO"
- board text removed: "SWO"

Commit message: Started layout
Parts:
- removed R3: 5k1, Resistor_SMD:R_0603_1608Metric
- removed SW1, SW2: SW_Push, Button_Switch_SMD:SW_Push_1P1T_NO_CK_KSC7xxJ
- added REF**: MountingHole_3.2mm_M3, MountingHole:MountingHole_3.2mm_M3, F.Cu at (109.0, 139.0)
- moved C35 406.5 mm to (84.6, 50.9)
- moved D12 406.5 mm to (87.8, 52.2)
- moved R22 406.5 mm to (84.6, 53.5)
- moved R24 406.5 mm to (90.9, 53.5)
- moved R26 406.5 mm to (90.9, 50.9)
- moved R42 391.5 mm to (80.1, 64.3), turned to 90 degrees
- moved R41 388.9 mm to (86.5, 70.6), turned to -90 degrees
- moved R40 388.4 mm to (80.1, 57.9), turned to -90 degrees
- moved D15 388.2 mm to (81.4, 61.1), turned to 0 degrees
- moved R44 388.2 mm to (82.7, 64.3), turned to 90 degrees
- moved C44 385.0 mm to (82.7, 57.9), turned to -90 degrees
- moved R45 384.7 mm to (90.3, 70.6), turned to 90 degrees
- moved R43 383.1 mm to (88.4, 70.6), turned to -90 degrees
- moved C46 382.5 mm to (90.9, 78.9), turned to 90 degrees
- moved U15 380.5 mm to (87.1, 76.3), turned to -90 degrees
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Connections:
- J1 pad B5: CAN+ -> CAN-
- J1 pad B6: CAN- -> CAN+
- U3 pad 44: /STM32/BOOT0 -> GND
- U3 pad 7: /STM32/NRST -> +3V3
Routing:
- net GND: track 2.61 -> 15.6 mm, vias 1 -> 6
- net Net-(R41-Pad2): track 0.00 -> 2.63 mm
- net Net-(R23-Pad2): track 0.00 -> 2.63 mm
- net Net-(R35-Pad2): track 0.00 -> 2.63 mm
- net Net-(R29-Pad2): track 0.00 -> 2.63 mm
- net Net-(R17-Pad2): track 0.00 -> 2.63 mm
- net Net-(R27-Pad1): track 0.00 -> 2.55 mm
- net Net-(R33-Pad1): track 0.00 -> 2.55 mm
- net Net-(R21-Pad1): track 0.00 -> 2.55 mm
- net Net-(R45-Pad1): track 0.00 -> 2.55 mm
- net Net-(R39-Pad1): track 0.00 -> 2.55 mm
- net Net-(R43-Pad2): track 0.00 -> 2.05 mm
- net Net-(R31-Pad2): track 0.00 -> 2.05 mm
- net Net-(R25-Pad2): track 0.00 -> 2.05 mm
- net Net-(R19-Pad2): track 0.00 -> 2.05 mm
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- added copper zone on In2.Cu, net +12V
- added copper zone on In2.Cu, net +3V3
- added copper zone on In1.Cu, net GND
- added copper zone on B.Cu, net H0
- added copper zone on B.Cu, net H1
- added copper zone on F.Cu, net H1
- added copper zone on B.Cu, net H2
- added copper zone on F.Cu, net H2
- added copper zone on B.Cu, net H3
- added copper zone on F.Cu, net H3
- added copper zone on B.Cu, net H4
- added copper zone on F.Cu, net H4
- added copper zone on B.Cu, net H5
- added copper zone on F.Cu, net H5
Other:
- board outline added: 82.4 x 100 mm

Commit message: Worked on layout
Parts:
- removed R46: 470, Resistor_SMD:R_0603_1608Metric
- added R3: 470, Resistor_SMD:R_0603_1608Metric, F.Cu at (137.3, 115.1)
- C1: value 100n -> 100uF; footprint Capacitor_SMD:C_0402_1005Metric -> Capacitor_SMD:CP_Elec_6.3x7.7
- C2: value 100uF -> 100n; footprint Capacitor_SMD:CP_Elec_6.3x7.7 -> Capacitor_SMD:C_0402_1005Metric
- D11: value 7V -> SSB43L; footprint Diode_SMD:D_MiniMELF -> Diode_SMD:D_SMB
- D16: value SP0502BAHT -> 7V; footprint Package_TO_SOT_SMD:SOT-23 -> Diode_SMD:D_MiniMELF
- D4: value 7V -> SP0502BAHT; footprint Diode_SMD:D_MiniMELF -> Package_TO_SOT_SMD:SOT-23
- D5: value SSB43L -> 7V; footprint Diode_SMD:D_SMB -> Diode_SMD:D_MiniMELF
- Q1, Q2, Q3, Q4, Q5, Q6: value IRLZ44N -> Si4162DY; footprint Package_TO_SOT_SMD:TO-263-2 -> Package_SO:SOIC-8_3.9x4.9mm_P1.27mm
- moved D4 85.4 mm to (137.9, 118.9), turned to 90 degrees
- moved C32 70.0 mm to (133.3, 87.6), turned to -90 degrees
- moved J3 68.5 mm to (74.2, 60.2), turned to 90 degrees
- moved R20 68.4 mm to (133.3, 94.0), turned to 90 degrees
- moved R16 66.5 mm to (130.8, 87.6), turned to -90 degrees
- moved C35 65.7 mm to (139.1, 87.6), turned to -90 degrees
- moved R18 64.9 mm to (130.8, 94.0), turned to 90 degrees
- moved R26 64.6 mm to (139.1, 94.0), turned to 90 degrees
- moved R22 62.2 mm to (136.5, 87.6), turned to -90 degrees
- moved R24 61.0 mm to (136.5, 94.0), turned to 90 degrees
- moved D15 58.9 mm to (112.4, 111.1)
- moved D12 58.8 mm to (132.1, 90.8), turned to 0 degrees
- moved D14 58.5 mm to (118.1, 111.1)
- moved R32 56.7 mm to (119.4, 114.3), turned to 90 degrees
- moved C17 56.3 mm to (102.2, 108.0)
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Connections:
- C1 pad 1: +3V3 -> +12V
- C2 pad 1: +12V -> +3V3
- D11 pad 1: Net-(D11-Pad1) -> +12V
- D11 pad 2: GND -> Net-(D11-Pad2)
- D16 pad 1: unconnected-(D16-Pad1) -> Net-(D16-Pad1)
- D16 pad 2: IO -> GND
- D4 pad 1: Net-(D4-Pad1) -> unconnected-(D4-Pad1)
- D4 pad 2: GND -> IO
- D5 pad 1: +12V -> Net-(D5-Pad1)
- D5 pad 2: Net-(D5-Pad2) -> GND
- F1 pad 1: Net-(D5-Pad2) -> Net-(D6-Pad2)
- F2 pad 1: Net-(D6-Pad2) -> Net-(D7-Pad2)
- F3 pad 1: Net-(D7-Pad2) -> Net-(D8-Pad2)
- F4 pad 1: Net-(D8-Pad2) -> Net-(D9-Pad2)
- F5 pad 1: Net-(D9-Pad2) -> Net-(D10-Pad2)
- F6 pad 1: Net-(D10-Pad2) -> Net-(D11-Pad2)
- Q1 pad 1: Net-(Q1-Pad1) -> GND
- Q1 pad 2: Net-(D5-Pad2) -> GND
- Q2 pad 1: Net-(Q2-Pad1) -> GND
- Q2 pad 2: Net-(D6-Pad2) -> GND
- Q3 pad 1: Net-(Q3-Pad1) -> GND
- Q3 pad 2: Net-(D7-Pad2) -> GND
- Q4 pad 1: Net-(Q4-Pad1) -> GND
- Q4 pad 2: Net-(D8-Pad2) -> GND
- Q5 pad 1: Net-(Q5-Pad1) -> GND
- Q5 pad 2: Net-(D9-Pad2) -> GND
- Q6 pad 1: Net-(Q6-Pad1) -> GND
- Q6 pad 2: Net-(D10-Pad2) -> GND
- R16 pad 2: Net-(D11-Pad1) -> Net-(D12-Pad1)
- R18 pad 2: Net-(D11-Pad1) -> Net-(D12-Pad1)
- R22 pad 2: Net-(D12-Pad1) -> Net-(D13-Pad1)
- R24 pad 2: Net-(D12-Pad1) -> Net-(D13-Pad1)
- R28 pad 2: Net-(D13-Pad1) -> Net-(D14-Pad1)
- R30 pad 2: Net-(D13-Pad1) -> Net-(D14-Pad1)
- R34 pad 2: Net-(D14-Pad1) -> Net-(D15-Pad1)
- R36 pad 2: Net-(D14-Pad1) -> Net-(D15-Pad1)
- R4 pad 2: Net-(D4-Pad1) -> Net-(D5-Pad1)
- R40 pad 2: Net-(D15-Pad1) -> Net-(D16-Pad1)
- R42 pad 2: Net-(D15-Pad1) -> Net-(D16-Pad1)
- R6 pad 2: Net-(D4-Pad1) -> Net-(D5-Pad1)
- U10 pad 5: Net-(Q6-Pad1) -> Net-(Q6-Pad4)
- U5 pad 5: Net-(Q1-Pad1) -> Net-(Q1-Pad4)
- U6 pad 5: Net-(Q2-Pad1) -> Net-(Q2-Pad4)
- U7 pad 5: Net-(Q3-Pad1) -> Net-(Q3-Pad4)
- U8 pad 5: Net-(Q4-Pad1) -> Net-(Q4-Pad4)
- U9 pad 5: Net-(Q5-Pad1) -> Net-(Q5-Pad4)
Routing:
- net GND: track 15.6 -> 155.5 mm, vias 6 -> 102
- net /STM32/UART_RX: track 0.00 -> 133.4 mm, vias 0 -> 4
- net /STM32/UART_TX: track 0.00 -> 130.3 mm, vias 0 -> 4
- net /High-side Channel 0/DEN: track 0.00 -> 127.3 mm, vias 0 -> 8
- net +12V: track 0.00 -> 98.6 mm, vias 253 -> 486
- net +3V3: track 0.00 -> 95.8 mm, vias 0 -> 19
- net /High-side Channel 5/Drive: track 0.00 -> 87.7 mm, vias 0 -> 4
- net /High-side Channel 0/Drive: track 0.00 -> 84.0 mm
- net CANTX: track 0.00 -> 80.2 mm, vias 0 -> 2
- net CANRX: track 0.00 -> 80.1 mm, vias 0 -> 2
- net /STM32/UU2: track 0.00 -> 75.3 mm, vias 0 -> 1
- net /STM32/UU0: track 0.00 -> 75.2 mm, vias 0 -> 1
- net /STM32/UU1: track 0.00 -> 71.7 mm, vias 0 -> 2
- net /STM32/UU3: track 0.00 -> 70.4 mm, vias 0 -> 1
- net /High-side Channel 0/Sense: track 0.00 -> 70.1 mm, vias 0 -> 2
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- added copper zone on F.Cu, net GND
- added copper zone on F.Cu, net Net-(D10-Pad2)
- added copper zone on F.Cu, net Net-(D11-Pad2)
- added copper zone on F.Cu, net Net-(D6-Pad2)
- added copper zone on F.Cu, net Net-(D7-Pad2)
- added copper zone on F.Cu, net Net-(D8-Pad2)
- added copper zone on F.Cu, net Net-(D9-Pad2)

Commit message: Worked on layout some more
Parts:
- renumbered REF** to H1
Routing:
- net GND: track 155.5 -> 145.0 mm, vias 102 -> 98
- net +12V: track 98.6 -> 94.9 mm, vias 486 -> 281
- net Net-(R35-Pad2): track 5.26 -> 2.53 mm
- net Net-(R41-Pad2): track 5.26 -> 2.53 mm
- net Net-(R29-Pad2): track 5.26 -> 2.53 mm
- net Net-(R17-Pad2): track 5.26 -> 2.53 mm
- net Net-(R23-Pad2): track 5.26 -> 2.53 mm
- net Net-(R45-Pad1): track 5.09 -> 2.55 mm
- net Net-(R39-Pad1): track 5.09 -> 2.55 mm
- net Net-(R33-Pad1): track 5.09 -> 2.55 mm
- net Net-(R21-Pad1): track 5.09 -> 2.55 mm
- net Net-(R27-Pad1): track 5.09 -> 2.55 mm
- net Net-(R43-Pad2): track 4.10 -> 2.01 mm
- net Net-(R37-Pad2): track 4.10 -> 2.01 mm
- net Net-(R31-Pad2): track 4.10 -> 2.01 mm
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Other:
- board text added: "L0"
- board text added: "L1"
- board text added: "L2"
- board text added: "L3"
- board text added: "L4"
- board text added: "L5"

Commit message: Finish layout (still needs memes)
Other:
- board text added: "+ -"
- board text added: "+12"
- board text added: "Bronco Racing BCM"
- board text added: "CAN"
- board text added: "H0"
- board text added: "H1"
- board text added: "H2"
- board text added: "H3"
- board text added: "H4"
- board text added: "H5"
- board text added: "IO0 IO1 IO2"
- board text added: "Jack LeFevre November 2022"
- board text added: "Rev. 5"
Changed lines of the file:
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@@
     )
   )
+  (gr_rect (start 136.9695 139.319) (end 148.9075 142.621) (layer "B.SilkS") (width 0.15) (fill none))
+  (gr_line (start 93.853 140.97) (end 94.488 140.97) (layer "B.SilkS") (width 0.15))
+  (gr_line (start 133.731 131.064) (end 135.001 131.064) (layer "B.SilkS") (width 0.15))
+  (gr_rect (start 82.042 132.588) (end 85.344 142.748) (layer "B.SilkS") (width 0.15) (fill none))
+  (gr_line (start 86.868 131.572) (end 88.646 131.572) (layer "B.SilkS") (width 0.15))
+  (gr_line (start 133.985 130.683) (end 134.747 130.683) (layer "B.SilkS") (width 0.15))
+  (gr_rect (start 137.033 132.461) (end 140.335 136.398) (layer "B.SilkS") (width 0.15) (fill none))
+  (gr_line (start 93.7895 134.62) (end 94.4245 134.62) (layer "B.SilkS") (width 0.15))
+  (gr_rect (start 132.715 132.461) (end 136.017 142.621) (layer "B.SilkS") (width 0.15) (fill none))
+  (gr_rect (start 86.106 132.588) (end 89.408 142.748) (layer "B.SilkS") (width 0.15) (fill none))
+  (gr_line (start 87.757 132.588) (end 87.757 131.572) (layer "B.SilkS") (width 0.15))
+  (gr_line (start 123.3805 141.097) (end 124.0155 141.097) (layer "B.SilkS") (width 0.15))
+  (gr_line (start 133.477 131.445) (end 135.255 131.445) (layer "B.SilkS") (width 0.15))
+  (gr_line (start 134.366 132.461) (end 134.366 131.445) (layer "B.SilkS") (width 0.15))
+  (gr_line (start 123.317 134.747) (end 123.952 134.747) (layer "B.SilkS") (width 0.15))
+  (gr_line (start 87.122 131.191) (end 88.392 131.191) (layer "B.SilkS") (width 0.15))
+  (gr_line (start 87.376 130.81) (end 88.138 130.81) (layer "B.SilkS") (width 0.15))
+  (gr_rect (start 141.224 132.461) (end 148.717 136.398) (layer "B.SilkS") (width 0.15) (fill none))
   (gr_line (start 67.832 143.442) (end 67.832 49.442) (layer "Edge.Cuts") (width 0.1))
   (gr_line (start 73.832 43.442) (end 67.832 49.442) (layer "Edge.Cuts") (width 0.1))
@@
     (effects (font (size 4 4) (thickness 0.6)) (justify mirror))
   )
+  (gr_text "+ -" (at 145.034 131.191) (layer "B.SilkS")
+    (effects (font (size 1.75 1.75) (thickness 0.3)) (justify mirror))
+  )
+  (gr_text "H3" (at 130.302 137.795 90) (layer "B.SilkS")
+    (effects (font (size 2 2) (thickness 0.3)) (justify mirror))
+  )
+  (gr_text "H5" (at 96.774 141.097) (layer "B.SilkS")
+    (effects (font (size 2 2) (thickness 0.3)) (justify mirror))
+  )
   (gr_text "L2" (at 92.075 95.25 90) (layer "B.SilkS")
     (effects (font (size 4 4) (thickness 0.6)) (justify mirror))
   )
+  (gr_text "+12" (at 83.82 129.286 90) (layer "B.SilkS")
+    (effects (font (size 2 2) (thickness 0.3)) (justify mirror))
+  )
+  (gr_text "L2" (at 75.438 131.318 90) (layer "B.SilkS")
+    (effects (font (size 2 2) (thickness 0.3)) (justify mirror))
+  )
+  (gr_text "L1" (at 71.12 137.922 90) (layer "B.SilkS")
+    (effects (font (size 2 2) (thickness 0.3)) (justify mirror))
+  )
+  (gr_text "H0" (at 96.901 134.747) (layer "B.SilkS")
+    (effects (font (size 2 2) (thickness 0.3)) (justify mirror))
+  )
+  (gr_text "H2" (at 130.302 131.191 90) (layer "B.SilkS")
+    (effects (font (size 2 2) (thickness 0.3)) (justify mirror))
+  )
   (gr_text "L4" (at 107.315 95.25 90) (layer "B.SilkS")
     (effects (font (size 4 4) (thickness 0.6)) (justify mirror))
   )
+  (gr_text "IO0 IO1 IO2" (at 142.875 138.049) (layer "B.SilkS")
+    (effects (font (size 1.5 1.25) (thickness 0.2)) (justify mirror))
+  )
+  (gr_text "L0" (at 71.12 131.318 90) (layer "B.SilkS")
+    (effects (font (size 2 2) (thickness 0.3)) (justify mirror))
+  )
+  (gr_text "L5" (at 79.502 137.922 90) (layer "B.SilkS")
+    (effects (font (size 2 2) (thickness 0.3)) (justify mirror))
+  )
   (gr_text "L5" (at 114.935 95.25 90) (layer "B.SilkS")
     (effects (font (size 4 4) (thickness 0.6)) (justify mirror))
@@
     (effects (font (size 4 4) (thickness 0.6)) (justify mirror))
   )
+  (gr_text "H4" (at 120.65 141.097) (layer "B.SilkS")
+    (effects (font (size 2 2) (thickness 0.3)) (justify mirror))
+  )
+  (gr_text "H1" (at 120.777 134.747) (layer "B.SilkS")
+    (effects (font (size 2 2) (thickness 0.3)) (justify mirror))
+  )
+  (gr_text "CAN" (at 145.034 129.032) (layer "B.SilkS")
+    (effects (font (size 2 2) (thickness 0.3)) (justify mirror))
+  )
+  (gr_text "L4" (at 79.502 131.318 90) (layer "B.SilkS")
+    (effects (font (size 2 2) (thickness 0.3)) (justify mirror))
+  )
+  (gr_text "L3" (at 75.438 137.922 90) (layer "B.SilkS")
+    (effects (font (size 2 2) (thickness 0.3)) (justify mirror))
+  )
+  (gr_text "+12" (at 138.811 129.159 90) (layer "B.SilkS")
+    (effects (font (size 2 2) (thickness 0.3)) (justify mirror))
+  )
   (gr_text "L0" (at 77.1144 95.25 90) (layer "B.SilkS")
     (effects (font (size 4 4) (thickness 0.6)) (justify mirror))
+  )
+  (gr_text "Rev. 5" (at 84.709 50.8) (layer "F.SilkS")
+    (effects (font (size 1.5 1.5) (thickness 0.3)))
+  )
+  (gr_text "Bronco Racing\nBCM" (at 72.263 49.657) (layer "F.SilkS")
+    (effects (font (size 2.5 2.5) (thickness 0.4)) (justify left))
+  )
+  (gr_text "Jack LeFevre\nNovember 2022" (at 109.982 58.039) (layer "F.SilkS")
+    (effects (font (size 2 2.3) (thickness 0.3)))
   )
   (segment (start 133.35 93.155) (end 132.105 93.155) (width 0.5) (layer "F.Cu") (net 1))
@@
     )
   )
+  (zone (net 0) (net_name "") (layer "B.Mask") (hatch edge 0.508)
+    (priority 1)
+    (connect_pads yes (clearance 0.25))
+    (min_thickness 0.254) (filled_areas_thickness no)
+    (fill yes (thermal_gap 0.508) (thermal_bridge_width 0.508))
+    (polygon
+      (pts
+        (xy 107.696 131.191)
+        (xy 99.314 131.191)
+        (xy 99.314 122.809)
+        (xy 107.696 122.809)
+      )
+    )
+  )
+  (zone (net 0) (net_name "") (layer "B.Mask") (hatch edge 0.508)
+    (priority 1)
+    (connect_pads yes (clearance 0.25))
+    (min_thickness 0.254) (filled_areas_thickness no)
+    (fill yes (thermal_gap 0.508) (thermal_bridge_width 0.508))
+    (polygon
+      (pts
+        (xy 128.016 130.429)
+        (xy 127.254 131.191)
+        (xy 119.634 131.191)
+        (xy 119.634 122.809)
+        (xy 128.016 122.809)
+      )
+    )
+  )
+  (zone (net 0) (net_name "") (layer "B.Mask") (hatch edge 0.508)
+    (priority 1)
+    (connect_pads yes (clearance 0.25))
+    (min_thickness 0.254) (filled_areas_thickness no)
+    (fill yes (thermal_gap 0.508) (thermal_bridge_width 0.508))
+    (polygon
+      (pts
+        (xy 97.536 131.191)
+        (xy 89.154 131.191)
+        (xy 89.154 122.809)
+        (xy 97.536 122.809)
+      )
+    )
+  )
+  (zone (net 0) (net_name "") (layer "B.Mask") (hatch edge 0.508)
+    (priority 1)
+    (connect_pads yes (clearance 0.25))
+    (min_thickness 0.254) (filled_areas_thickness no)
+    (fill yes (thermal_gap 0.508) (thermal_bridge_width 0.508))
+    (polygon
+      (pts
+        (xy 130.556 111.252)
+        (xy 122.174 111.252)
+        (xy 122.174 102.87)
+        (xy 130.556 102.87)
+      )
+    )
+  )
+  (zone (net 0) (net_name "") (layer "B.Mask") (hatch edge 0.508)
+    (priority 1)
+    (connect_pads yes (clearance 0.25))
+    (min_thickness 0.254) (filled_areas_thickness no)
+    (fill yes (thermal_gap 0.508) (thermal_bridge_width 0.508))
+    (polygon
+      (pts
+        (xy 117.856 131.191)
+        (xy 109.474 131.191)
+        (xy 109.474 122.809)
+        (xy 117.856 122.809)
+      )
+    )
+  )
+  (zone (net 0) (net_name "") (layer "B.Mask") (hatch edge 0.508)
+    (priority 1)
+    (connect_pads yes (clearance 0.25))
+    (min_thickness 0.254) (filled_areas_thickness no)
+    (fill yes (thermal_gap 0.508) (thermal_bridge_width 0.508))
+    (polygon
+      (pts
+        (xy 140.716 111.506)
+        (xy 132.588 111.506)
+        (xy 132.334 111.252)
+        (xy 132.334 103.124)
+        (xy 140.716 103.124)
+      )
+    )
+  )
+  (group "" (id 4b904132-7a5e-4d9f-b043-8a8656d9221b)
+    (members
+      4a13f84d-4a2f-49fc-9da2-758610fbdd62
+      83eb58fd-6269-4137-9e2a-3b89312a1d4c
+      8ab391ba-73fd-4782-ac92-8d0e8bdb18d9
+      c43e58c4-4317-4fff-ab84-9473a87d9f4d
+      c57009c8-f99a-4783-9242-c00e291cb1e8
+    )
+  )
+  (group "" (id 8b4166aa-292a-4e49-b546-202970e84035)
+    (members
+      7c3a71b1-6d74-4269-9594-4892f9a83800
+      922ad0d1-b159-4293-b1b9-dcd4a5edd6d9
+      935dc562-3532-4a6f-a81d-423757df13c5
+      ea4d6f4b-0f66-47dd-949a-308ceb6a91b3
+      f1379cb5-7a8c-4fac-be6e-b3b70b1c2fe0
+    )
+  )

Commit message: Fixed ERC
Connections:
- J3 pad 11: /STM32/UU8 -> unconnected-(J3-Pad11)
