File: pcb/PCB.kicad_pcb (KiCad board)
At the start: 4 copper layers, 82.4 x 100 mm, 141 parts, among them J1 DTM1312PA12PBR008, J2 TC2030, J3 Conn_02x08_Top_Bottom, J4 JST B04B-XASK, Q1 Si4162DY, Q2 Si4162DY, Q3 Si4162DY, Q4 Si4162DY, Q5 Si4162DY, Q6 Si4162DY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

Commit message: Bottom text
Other:
- board text added: "BOTTOM TEXT"
Changed lines of the file:
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@@
     (effects (font (size 2 2) (thickness 0.3)) (justify mirror))
+  )
+  (gr_text "BOTTOM TEXT" (at 109.347 79.883) (layer "B.SilkS")
+    (effects (font (size 7 7) (thickness 1.2)) (justify mirror))
   )
   (gr_text "+12" (at 138.811 129.159 90) (layer "B.SilkS")

Commit message: Disconnected NRESET
Connections:
- U3 pad 7: +3V3 -> unconnected-(U3-Pad7)
Routing:
- net +3V3: track 83.3 -> 80.6 mm
Changed lines of the file:
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@@
   (net 140 "Net-(Q5-Pad4)")
   (net 141 "Net-(Q6-Pad4)")
+  (net 142 "unconnected-(U3-Pad7)")
   (footprint "Capacitor_SMD:C_0805_2012Metric" (layer "F.Cu")
     (at 91.12 66.538)
@@
       (net 8 "/STM32/HSE_IN") (pinfunction "PD1") (pintype "input"))
     (pad "7" smd roundrect (at -4.1625 0.25) (size 1.475 0.3) (layers "F.Cu" "F.Paste" "F.Mask") (roundrect_rratio 0.25)
-      (net 2 "+3V3") (pinfunction "NRST") (pintype "input"))
+      (net 142 "unconnected-(U3-Pad7)") (pinfunction "NRST") (pintype "input+no_connect"))
     (pad "8" smd roundrect (at -4.1625 0.75) (size 1.475 0.3) (layers "F.Cu" "F.Paste" "F.Mask") (roundrect_rratio 0.25)
       (net 1 "GND") (pinfunction "VSSA") (pintype "power_in"))
@@
   (segment (start 139.54 75.278) (end 141.224 75.278) (width 1) (layer "F.Cu") (net 2))
   (segment (start 129.255 59.845) (end 129.07 59.66) (width 0.2) (layer "F.Cu") (net 2))
-  (segment (start 131.54 61.21) (end 130.175 59.845) (width 0.2) (layer "F.Cu") (net 2))
   (segment (start 144.09 57.94) (end 144.12 57.91) (width 0.2) (layer "F.Cu") (net 2))
   (segment (start 129.68 67.945) (end 130.805 67.945) (width 0.5) (layer "F.Cu") (net 2))
@@
   (segment (start 133.61 76.714) (end 133.604 76.708) (width 1) (layer "F.Cu") (net 2))
   (segment (start 139.275 67.04) (end 139.545 67.31) (width 0.2) (layer "F.Cu") (net 2))
-  (segment (start 132.3625 61.21) (end 131.54 61.21) (width 0.2) (layer "F.Cu") (net 2))
   (segment (start 142.654 75.278) (end 141.224 75.278) (width 1) (layer "F.Cu") (net 2))
   (segment (start 142.605 58.21) (end 142.875 57.94) (width 0.2) (layer "F.Cu") (net 2))

Commit message: Udpate date/revision of BCM
Other:
- board text added: "Jack LeFevre March 2023"
- board text removed: "Jack LeFevre November 2022"
Changed lines of the file:
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@@
     (effects (font (size 2.5 2.5) (thickness 0.4)) (justify left))
   )
-  (gr_text "Jack LeFevre\nNovember 2022" (at 109.982 58.039) (layer "F.SilkS")
+  (gr_text "Jack LeFevre\nMarch 2023" (at 109.982 58.039) (layer "F.SilkS")
     (effects (font (size 2 2.3) (thickness 0.3)))
   )
