File: pcb/highside.kicad_sch (KiCad schematic)
At the start: 11 parts, among them U4 BTS7004-1EPP

Commit message: Worked on layout
Parts:
- renumbered D4 to D5
Changed lines of the file:
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@@
   (symbol (lib_id "Device:D_Zener") (at 146.05 74.93 270) (unit 1)
     (in_bom yes) (on_board yes) (fields_autoplaced)
-    (property "Reference" "D4" (id 0) (at 148.59 73.6599 90)
+    (property "Reference" "D5" (id 0) (at 148.59 73.6599 90)
       (effects (font (size 1.27 1.27)) (justify left))
     )
@@
   (symbol (lib_id "power:GND") (at 176.53 86.36 0) (unit 1)
     (in_bom yes) (on_board yes) (fields_autoplaced)
-    (property "Reference" "#PWR033" (id 0) (at 176.53 92.71 0)
+    (property "Reference" "#PWR039" (id 0) (at 176.53 92.71 0)
       (effects (font (size 1.27 1.27)) hide)
     )
@@
   (symbol (lib_id "power:+12V") (at 143.51 100.33 0) (unit 1)
     (in_bom yes) (on_board yes) (fields_autoplaced)
-    (property "Reference" "#PWR030" (id 0) (at 143.51 104.14 0)
+    (property "Reference" "#PWR036" (id 0) (at 143.51 104.14 0)
       (effects (font (size 1.27 1.27)) hide)
     )
@@
   (symbol (lib_id "power:+12V") (at 176.53 54.61 0) (unit 1)
     (in_bom yes) (on_board yes) (fields_autoplaced)
-    (property "Reference" "#PWR032" (id 0) (at 176.53 58.42 0)
+    (property "Reference" "#PWR038" (id 0) (at 176.53 58.42 0)
       (effects (font (size 1.27 1.27)) hide)
     )
@@
   (symbol (lib_id "power:PWR_FLAG") (at 176.53 72.39 270) (unit 1)
     (in_bom yes) (on_board yes) (fields_autoplaced)
-    (property "Reference" "#FLG0101" (id 0) (at 178.435 72.39 0)
+    (property "Reference" "#FLG04" (id 0) (at 178.435 72.39 0)
       (effects (font (size 1.27 1.27)) hide)
     )
@@
   (symbol (lib_id "power:GND") (at 143.51 107.95 0) (unit 1)
     (in_bom yes) (on_board yes) (fields_autoplaced)
-    (property "Reference" "#PWR031" (id 0) (at 143.51 114.3 0)
-      (effects (font (size 1.27 1.27)) hide)
-    )
+    (property "Reference" "#PWR037" (id 0) (at 143.51 114.3 0)
+      (effects (font (size 1.27 1.27)) hide)
+    )
