File: pcb/lowside.kicad_sch (KiCad schematic)
At the start: 7 parts, among them Q1 IRLZ44N, U5 MCP1416

Commit message: Worked on layout
Parts:
- removed Q1: IRLZ44N, Package_TO_SOT_SMD:TO-263-2, symbol Transistor_FET:IRLZ44N
- added Q6: Si4162DY, Package_SO:SOIC-8_3.9x4.9mm_P1.27mm, symbol Transistor_FET:Si4162DY
- renumbered D5 to D6
Connections:
- net GND: now also Q6.1 (S), Q6.2 (S), Q6.3 (S)
- net at D6.2 (A), F1.1: now also Q6.5 (D), Q6.6 (D), Q6.7 (D), Q6.8 (D)
- net at U5.5 (OUT): now also Q6.4 (G)
Changed lines of the file:
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@@
   (symbol (lib_id "power:+12V") (at 160.02 78.74 0) (unit 1)
     (in_bom yes) (on_board yes)
-    (property "Reference" "#PWR036" (id 0) (at 160.02 82.55 0)
+    (property "Reference" "#PWR042" (id 0) (at 160.02 82.55 0)
       (effects (font (size 1.27 1.27)) hide)
     )
@@
   (symbol (lib_id "Device:D_Schottky") (at 160.02 82.55 270) (unit 1)
     (in_bom yes) (on_board yes) (fields_autoplaced)
-    (property "Reference" "D5" (id 0) (at 162.56 80.9624 90)
+    (property "Reference" "D6" (id 0) (at 162.56 80.9624 90)
       (effects (font (size 1.27 1.27)) (justify left))
     )
@@
     (pin "5")
   )
+  (symbol (lib_id "Transistor_FET:Si4162DY") (at 157.48 91.44 0) (unit 1)
+    (in_bom yes) (on_board yes) (fields_autoplaced)
+    (property "Reference" "Q6" (id 0) (at 163.83 90.1699 0)
+      (effects (font (size 1.27 1.27)) (justify left))
+    )
+    (property "Value" "Si4162DY" (id 1) (at 163.83 92.7099 0)
+      (effects (font (size 1.27 1.27)) (justify left))
+    )
+    (property "Footprint" "Package_SO:SOIC-8_3.9x4.9mm_P1.27mm" (id 2) (at 162.56 93.98 0)
+      (effects (font (size 1.27 1.27)) (justify left) hide)
+    )
+    (property "Datasheet" "http://www.vishay.com/docs/68967/si4162dy.pdf" (id 3) (at 157.48 91.44 0)
+      (effects (font (size 1.27 1.27)) (justify left) hide)
+    )
+    (pin "1")
+    (pin "2")
+    (pin "3")
+    (pin "4")
+    (pin "5")
+    (pin "6")
+    (pin "7")
+    (pin "8")
+  )
   (symbol (lib_id "power:+12V") (at 147.32 118.11 0) (unit 1)
     (in_bom yes) (on_board yes)
-    (property "Reference" "#PWR034" (id 0) (at 147.32 121.92 0)
+    (property "Reference" "#PWR040" (id 0) (at 147.32 121.92 0)
       (effects (font (size 1.27 1.27)) hide)
     )
@@
     (pin "1")
   )
-  (symbol (lib_id "Transistor_FET:IRLZ44N") (at 157.48 91.44 0) (unit 1)
-    (in_bom yes) (on_board yes) (fields_autoplaced)
-    (property "Reference" "Q1" (id 0) (at 163.83 90.1699 0)
-      (effects (font (size 1.27 1.27)) (justify left))
-    )
-    (property "Value" "IRLZ44N" (id 1) (at 163.83 92.7099 0)
-      (effects (font (size 1.27 1.27)) (justify left))
-    )
-    (property "Footprint" "Package_TO_SOT_SMD:TO-263-2" (id 2) (at 163.83 93.345 0)
-      (effects (font (size 1.27 1.27) italic) (justify left) hide)
-    )
-    (property "Datasheet" "http://www.irf.com/product-info/datasheets/data/irlz44n.pdf" (id 3) (at 157.48 91.44 0)
-      (effects (font (size 1.27 1.27)) (justify left) hide)
-    )
-    (pin "1")
-    (pin "2")
-    (pin "3")
-  )
   (symbol (lib_id "power:GND") (at 147.32 125.73 0) (unit 1)
     (in_bom yes) (on_board yes) (fields_autoplaced)
-    (property "Reference" "#PWR035" (id 0) (at 147.32 132.08 0)
+    (property "Reference" "#PWR041" (id 0) (at 147.32 132.08 0)
       (effects (font (size 1.27 1.27)) hide)
     )
@@
   (symbol (lib_id "power:GND") (at 160.02 101.6 0) (unit 1)
     (in_bom yes) (on_board yes) (fields_autoplaced)
-    (property "Reference" "#PWR037" (id 0) (at 160.02 107.95 0)
+    (property "Reference" "#PWR043" (id 0) (at 160.02 107.95 0)
       (effects (font (size 1.27 1.27)) hide)
     )

Commit message: Worked on layout some more
Parts:
- renumbered Q6 to Q1
Changed lines of the file:
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@@
   (symbol (lib_id "Transistor_FET:Si4162DY") (at 157.48 91.44 0) (unit 1)
     (in_bom yes) (on_board yes) (fields_autoplaced)
-    (property "Reference" "Q6" (id 0) (at 163.83 90.1699 0)
+    (property "Reference" "Q1" (id 0) (at 163.83 90.1699 0)
       (effects (font (size 1.27 1.27)) (justify left))
     )
