File: pcb/PCB.kicad_sch (KiCad schematic)
At the start: 19 parts, among them J1 DTM1312PA12PBR008, J4 JST B04B-XASK, U1 SN65HVD230, U2 LF33_TO252

Commit message: Bottom text
Parts:
- J1: footprint TE_DTM1312PA12PBR008 -> DTM13-12PA-12PB:TE_DTM1312PA12PBR008
Changed lines of the file:
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@@
     (property "Reference" "J1" (id 0) (at 222.25 67.31 0))
     (property "Value" "DTM1312PA12PBR008" (id 1) (at 222.25 69.85 0))
-    (property "Footprint" "TE_DTM1312PA12PBR008" (id 2) (at 222.25 87.63 0)
+    (property "Footprint" "DTM13-12PA-12PB:TE_DTM1312PA12PBR008" (id 2) (at 222.25 87.63 0)
       (effects (font (size 1.27 1.27)) (justify left bottom) hide)
     )
@@
     )
     (path "/d6bde4d9-ffb7-4d4e-ae84-524e1254604a"
-      (reference "J1") (unit 1) (value "DTM1312PA12PBR008") (footprint "TE_DTM1312PA12PBR008")
+      (reference "J1") (unit 1) (value "DTM1312PA12PBR008") (footprint "DTM13-12PA-12PB:TE_DTM1312PA12PBR008")
     )
     (path "/1d08d960-24a6-461a-b4f3-543e0f014558/86b61b36-28e1-4d1c-9f8e-bc6fc9a33198"
